File: Button Mainboard Interface/Button Mainboard Interface.kicad_pcb (KiCad board)
At the start: 2 copper layers, 42 x 50.2 mm, 25 parts, among them J1 Conn_01x02, J10 Conn_01x02, J100 Conn_02x07_Odd_Even, J11 Conn_01x02, J12 Conn_01x02, J2 Conn_01x02, J3 Conn_01x02, J4 Conn_01x02, J5 Conn_01x02, J6 Conn_01x02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

Commit message: Released PCB
Other:
- board text added: "REV X0"
Changed lines of the file:
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@@
 			(outputformat 1)
 			(mirror no)
-			(drillshape 1)
+			(drillshape 0)
 			(scaleselection 1)
-			(outputdirectory "")
+			(outputdirectory "Fabrication_data_Button_Mainboard_Interface")
 		)
 	)
@@
 		(layer "Edge.Cuts")
 	)
+	(gr_text "REV X0"
+		(at 141.15 85.1 90)
+		(layer "F.SilkS")
+		(effects
+			(font
+				(size 1.5 1.5)
+				(thickness 0.3)
+				(bold yes)
+			)
+			(justify left bottom)
+		)
+	)
 	(gr_text "Button Breakout\nTo Analog Board\nCMSC 2026\nNathan Ford"
