File: Button Mainboard Interface/Button Mainboard Interface.kicad_sch (KiCad schematic)
At the start: 25 parts, among them J1 Conn_01x02, J10 Conn_01x02, J100 Conn_02x07_Odd_Even, J11 Conn_01x02, J12 Conn_01x02, J2 Conn_01x02, J3 Conn_01x02, J4 Conn_01x02, J5 Conn_01x02, J6 Conn_01x02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

Commit message: Released PCB
Other:
- company: (none) -> CMSC
- title: (none) -> Button Mainboard Interface
Changed lines of the file:
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@@
 	(generator_version "9.0")
 	(paper "A4")
+	(title_block
+		(title "Button Mainboard Interface")
+		(date "2026-01-15")
+		(rev "X0")
+		(company "CMSC")
+		(comment 1 "Drawn 1-15-26 by NF")
+		(comment 2 "Released 1-15-26 by NF")
+	)
 	(junction
 		(at 49.53 88.9)
